File: header.sch (KiCad schematic (older format))
At the start: 33 parts, among them Q3 Q_NMOS_GSD, Q4 Q_NMOS_GSD, U10 MAX40200AUK, U11 MAX40200AUK, U12 TXS0108EPW, U13 MAX11614, U14 TXS0108EPW, Y1 ECS-3225S33-500-FN-TR

Commit message: Board design completed Revision 1
Connections:
- net FPGA_INO_MISO: now also U12.4 (A3); no longer U12.5 (A4)
- net FPGA_INO_RX: now also U14.8 (A7); no longer U14.9 (A8)
- net FPGA_INO_SCK: now also U12.5 (A4); no longer U12.4 (A3)
- net FPGA_INO_TX: now also U14.9 (A8); no longer U14.8 (A7)
- net INO_MISO: now also U12.17 (B3); no longer U12.16 (B4)
- net INO_RX: now also U14.13 (B7); no longer U14.12 (B8)
- net INO_SCK: now also U12.16 (B4); no longer U12.17 (B3)
- net INO_TX: now also U14.12 (B8); no longer U14.13 (B7)
Changed lines of the file:
@@
 Wire Wire Line
 	8025 1750 7625 1750
+Text Label 8025 1550 2    50   ~ 0
+INO_MISO
+Wire Wire Line
+	8025 1650 7625 1650
 Text Label 8025 1650 2    50   ~ 0
-INO_MISO
-Wire Wire Line
-	8025 1650 7625 1650
-Text Label 8025 1550 2    50   ~ 0
 INO_SCK
 Wire Wire Line
@@
 Wire Wire Line
 	9875 775  9875 850
-Text Label 10775 1950 2    50   ~ 0
-INO_RX
 Wire Wire Line
 	10775 1950 10375 1950
-Text Label 10775 1850 2    50   ~ 0
-INO_TX
 Wire Wire Line
 	10775 1850 10375 1850
@@
 Text HLabel 6825 1250 0    50   Input ~ 0
 OE1
-Text HLabel 9575 1850 0    50   Input ~ 0
+Text HLabel 9575 1950 0    50   Input ~ 0
 FPGA_INO_TX
-Text HLabel 9575 1950 0    50   Output ~ 0
+Text HLabel 9575 1850 0    50   Output ~ 0
 FPGA_INO_RX
 Text HLabel 6825 1350 0    50   BiDi ~ 0
 FPGA_INO_SCL
+Text HLabel 6825 1650 0    50   BiDi ~ 0
+FPGA_INO_SCK
 Text HLabel 6825 1550 0    50   BiDi ~ 0
-FPGA_INO_SCK
-Text HLabel 6825 1650 0    50   BiDi ~ 0
 FPGA_INO_MISO
 Text HLabel 6825 1750 0    50   BiDi ~ 0
@@
 Wire Wire Line
 	7750 3475 7750 3450
+Text Label 10775 1850 2    50   ~ 0
+INO_RX
+Text Label 10775 1950 2    50   ~ 0
+INO_TX
 $EndSCHEMATC
